File: hardware_design/motherboard/ESP32_Interfaces_Board_v02b1.kicad_pcb (KiCad board)
At the start: 2 copper layers, 89.1 x 84.5 mm, 53 parts, among them J1 32K145-400L5, P1 Header 8, P2 Header 2X2, P3 Header 6, U1 ESP32_Devkit_V1, U2 JMD0.96-12864, U3 Button1, U4 Button2, U5 FM-B2020RGBA-HG, U6 ATGM336H-GPS

Commit message: pcie routed
Parts:
- added ?: , , F.Cu at (113.6, 67.2)
- added ?: , , F.Cu at (113.6, 91.4)
- added REF**: BUS_PCI_Express_Mini_Dual-small-pad, danman:BUS_PCI_Express_Mini_Dual-small-pad, F.Cu at (161.7, 79.3)
Routing:
- net VCC3V3: track 133.7 -> 173.3 mm, vias 3 -> 4
- net NSS: track 67.2 -> 99.7 mm
- net MISO: track 75.4 -> 107.9 mm
- net SCL: track 110.7 -> 142.3 mm, vias 0 -> 1
- net MOSI: track 68.6 -> 99.2 mm, vias 1 -> 3
- net SDA: track 88.7 -> 116.2 mm
- net SCK: track 79.9 -> 105.5 mm, vias 1 -> 2
- net NRESET: track 62.1 -> 86.7 mm
- net 1PPS: track 97.8 -> 115.1 mm
- net GND: track 0.00 -> 3.11 mm, vias 608 -> 587
